File: PCB/IIT_5dof_arm/IIT_5dof_arm.kicad_sch (KiCad schematic)
At the start: 101 parts, among them J1 Barrel_Jack_Switch, J10 Conn_01x06, J11 Conn_01x06, J12 Conn_01x06, J13 Conn_01x06, J14 Conn_02x13_Top_Bottom, J2 Conn_01x04, J3 Conn_01x04, J4 Conn_02x10_Counter_Clockwise, J5 Conn_01x04, J6 Conn_02x13_Top_Bottom, J7 Conn_01x06, J8 Conn_02x10_Counter_Clockwise, J9 Conn_01x06, Q1 2N7000, Q2 2N7000, SW1 SW_MAIN, SW10 SW_Push, SW11 SW_Push, SW12 SW_Push, SW13 SW_Push, SW14 SW_Push, SW15 SW_MOT, SW2 SW_Push, SW3 RotaryEncoder_Switch, SW4 SW_Push, SW5 SW_Push, SW6 SW_Push, SW7 SW_Push, SW8 SW_Push, SW9 SW_Push, U5 XL8574T, U6 XL8574T, U7 XL8574T

Commit message: Separated UI to ATmega controller
Parts:
- removed D18, D19: LED, LED_THT:LED_D5.0mm, symbol Device:LED
- removed J2, J3: Conn_01x04, Connector_Molex:Molex_KK-254_AE-6410-04A_1x04_P2.54mm_Vertical, symbol Connector_Generic:Conn_01x04
- removed J4, J8: Conn_02x10_Counter_Clockwise, Connector_IDC:IDC-Header_2x10_P2.54mm_Vertical, symbol Connector_Generic:Conn_02x10_Counter_Clockwise
- removed U6, U7: XL8574T, Package_SO:SOIC-16W_7.5x10.3mm_P1.27mm, symbol Interface_Expansion:PCF8574
- added C2, C3: 22pF, symbol Device:C
- added C4, C5: 1uF, symbol Device:C
- added C6, C7, C9: 100nF, symbol Device:C
- added C8: 4.7uF, symbol Device:C_Polarized
- added J15, J3: Conn_01x03, Connector_Molex:Molex_KK-254_AE-6410-03A_1x03_P2.54mm_Vertical, symbol Connector_Generic:Conn_01x03
- added J2: Conn_02x03_Counter_Clockwise, symbol Connector_Generic:Conn_02x03_Counter_Clockwise
- added J4, J8: Conn_01x04, Connector_Molex:Molex_KK-254_AE-6410-04A_1x04_P2.54mm_Vertical, symbol Connector_Generic:Conn_01x04
- added R17, R18, R46, R47, R48: 180, Resistor_SMD:R_0805_2012Metric_Pad1.20x1.40mm_HandSolder, symbol Device:R
- added R44, R45, R49, R50, R51: 390, Resistor_SMD:R_0805_2012Metric_Pad1.20x1.40mm_HandSolder, symbol Device:R
- added R52: 10k, Resistor_SMD:R_0805_2012Metric_Pad1.20x1.40mm_HandSolder, symbol Device:R
- added SW16: SW_Push, Connector_Molex:Molex_KK-254_AE-6410-02A_1x02_P2.54mm_Vertical, symbol Switch:SW_Push
- added U8: ATmega48-20A, Package_QFP:TQFP-32_7x7mm_P0.8mm, symbol MCU_Microchip_ATmega:ATmega48-20A
- added Y1: 16MHz, symbol Device:Crystal
- R39: value 65 -> 180
- R40: value 65 -> 390
Connections:
- net Mot1_BUTT_A is gone; now on net ~{Fault}_34: U5.11 (P6)
- net Mot1_BUTT_B is gone; now on net ~{Fault}_56: U5.12 (P7)
- net UIPanel_+3V3 is gone; now on net UIPanel_+5V: J5.1 (Pin_1), R33.2, R34.2, SW3.S1
- net UI_Enc_A is gone; now on net mot4_B: U4.10 (GPIO26/ADC19/DAC2)
- net UI_Enc_B is gone; now on net mot3_A: U4.11 (GPIO27/ADC17/TOUCH7)
- net +3V3: now also U5.16 (VDD)
- net +5V: now also J8.1 (Pin_1); no longer U5.16 (VDD)
- net GND: now also R40.1, J8.4 (Pin_4), R44.1, R45.1, R49.1, R50.1, R51.1
- net Mot1_LIMIT_IN: now also R17.1; no longer U5.4 (P0)
- net Mot2_LIMIT_IN: now also R18.1; no longer U5.5 (P1)
- net Mot3_LIMIT_IN: now also R39.1; no longer U5.6 (P2)
- net Mot4_LIMIT_IN: now also R46.1; no longer U5.7 (P3)
- net Mot5_LIMIT_IN: now also R47.1; no longer U5.9 (P4)
- net Mot6_LIMIT_IN: now also R48.1; no longer U5.10 (P5)
- net SCL_3v3: now also U5.14 (SCL); no longer Q1.1 (S), R16.2, R37.2
- net SDA_3v3: now also U5.15 (SDA); no longer Q2.1 (S), R15.2, R38.2
- net UIPanel_+5V: now also C4.1, C5.1, C8.1, J15.1 (Pin_1), J2.6 (Pin_6), J3.1 (Pin_1), J4.1 (Pin_1), R52.2, U8.18 (AVCC), U8.4 (VCC), U8.6 (VCC)
- net UIPanel_BUTT1A: now also U8.12 (PB0)
- net UIPanel_BUTT1B: now also U8.23 (PC0)
- net UIPanel_BUTT2A: now also U8.13 (PB1)
- net UIPanel_BUTT2B: now also U8.24 (PC1)
- net UIPanel_BUTT3A: now also U8.14 (PB2)
- net UIPanel_BUTT3B: now also U8.25 (PC2)
- net UIPanel_BUTT4B: now also U8.26 (PC3); no longer R26.2, SW9.2
- net UIPanel_BUTT5B: now also U8.2 (PD4); no longer R27.2, SW10.2
- net UIPanel_BUTT6B: now also U8.9 (PD5); no longer R28.2, SW11.2
- net UIPanel_Enc_A: now also C7.1, U8.32 (PD2)
- net UIPanel_Enc_B: now also C6.1, U8.1 (PD3)
- net UIPanel_Enc_BUTT: now also U8.10 (PD6)
- net UIPanel_GND: now also C2.2, C3.1, C4.2, C5.2, C6.2, C7.2, C8.2, C9.2, J15.3 (Pin_3), J2.4 (Pin_4), J3.3 (Pin_3), J4.4 (Pin_4), SW16.2, U8.21 (GND), U8.3 (GND), U8.5 (GND)
- net UIPanel_SCL: now also U8.28 (PC5)
- net UIPanel_SDA: now also U8.27 (PC4)
- net mot3_A: no longer U4.27 (GPIO16/RX2)
- net mot4_B: no longer U4.28 (GPIO17/TX2)
- net ~{Fault}_12: now also U4.9 (GPIO25/ADC18/DAC1)
- net at BZ1.1 (+): now also U8.11 (PD7); no longer U4.9 (GPIO25/ADC18/DAC1)
- net Reserved_LED1 renamed Mot3_LIMIT
- net Mot3_LIMIT: now also U5.6 (P2), R45.2
- net Reserved_LED2 renamed Mot1_LIMIT
- net Mot1_LIMIT: now also U5.4 (P0), R17.2
- net SCL_5v renamed UI_TX_5v
- net UI_TX_5v: now also J8.2 (Pin_2); no longer U5.14 (SCL)
- net SDA_5v renamed UI_RX_5v
- net UI_RX_5v: now also J8.3 (Pin_3); no longer U5.15 (SDA)
- new net: C9.1, U8.20 (AREF)
- new net Mot2_LIMIT: R18.2, R44.2, U5.5 (P1)
- new net Mot4_LIMIT: R46.2, R49.2, U5.7 (P3)
- new net Mot5_LIMIT: R47.2, R50.2, U5.9 (P4)
- new net Mot6_LIMIT: R48.2, R51.2, U5.10 (P5)
- new net UIPanel_ADC1: J3.2 (Pin_2), U8.19 (ADC6)
- new net UIPanel_ADC2: J15.2 (Pin_2), U8.22 (ADC7)
- new net UIPanel_BUTT4A: J2.5 (Pin_5), R26.2, SW9.2, U8.15 (PB3)
- new net UIPanel_BUTT5A: J2.1 (Pin_1), R27.2, SW10.2, U8.16 (PB4)
- new net UIPanel_BUTT6A: J2.2 (Pin_2), R28.2, SW11.2, U8.17 (PB5)
- new net UIPanel_RX: J4.2 (Pin_2), U8.30 (PD0)
- new net UIPanel_TX: J4.3 (Pin_3), U8.31 (PD1)
- new net UIPanel_reset: J2.3 (Pin_3), R52.1, SW16.1, U8.29 (~{RESET}/PC6)
- new net UI_RX_3v3: Q2.1 (S), R15.2, R38.2, U4.27 (GPIO16/RX2)
- new net UI_TX_3v3: Q1.1 (S), R16.2, R37.2, U4.28 (GPIO17/TX2)
- new net XTAL1: C2.1, U8.7 (XTAL1/PB6), Y1.2
- new net XTAL2: C3.2, U8.8 (XTAL2/PB7), Y1.1
Other:
- note added: "Motor power feedback LED"
- note added: "Port expanding"
- note added: "UART feedback LED"
- note added: "UART level shifting"
- note removed: "Ha csak 2V-3V-ig megy lehet, hogy a limiteken kívül le lehetne vinni 3v3-ra"
- note removed: "I2C feedback LED"
- note removed: "I2C level shifting"
- note removed: "Open drainek a port extenderek -> elvileg nem kell 5V-ig felhúzni"
- note removed: "Port extender interrupt level shifting"
- note removed: "Port extending"
- note removed: "Power feedback LED"
- moved on the sheet: BZ1, C1, D10, D11, D12, D13, D14, D15, D16, D2, D3, D5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

Commit message: Switch UART level shift to 2in1 fet, resistor values corrected
Parts:
- removed Q1, Q2: 2N7000, Package_TO_SOT_THT:TO-92_Inline, symbol Transistor_FET:2N7000
- added Q3: FDG6335N, Package_TO_SOT_SMD:SOT-363_SC-70-6, symbol Transistor_FET:FDG6335N
- R13, R14, R15, R16: value 2k2 -> 10k
- R20, R21, R22, R23, R24, R25, R26, R27, R28, R29, R30, R31, R35, R37, R38: value 165 -> 220
Connections:
- net +3V3: now also Q3.2 (G), Q3.5 (G)
- net UIPanel_BUTT4A: no longer J2.5 (Pin_5), U8.15 (PB3)
- net UIPanel_BUTT5A: no longer J2.1 (Pin_1), U8.16 (PB4)
- net UIPanel_BUTT6A: no longer J2.2 (Pin_2), U8.17 (PB5)
- net UI_RX_3v3: now also Q3.4 (S)
- net UI_RX_5v: now also Q3.3 (D)
- net UI_TX_3v3: now also Q3.1 (S)
- net UI_TX_5v: now also Q3.6 (D)
- new net UIPanel_BUTT4A__UIPanel_Prog_MOSI: J2.5 (Pin_5), U8.15 (PB3)
- new net UIPanel_BUTT5A__UIPanel_Prog_MISO: J2.1 (Pin_1), U8.16 (PB4)
- new net UIPanel_BUTT6A__UIPanel_Prog_SCK: J2.2 (Pin_2), U8.17 (PB5)
Other:
- note added: "Connection to robot interface"
- note added: "Programming with: https://github.com/MCUdude/MiniCore"
- note added: "Robot arm interface panel"
- note added: "User interface panel"
- note removed: "I/O connections"
- note removed: "I/O connections with robot arm"
- note removed: "User interface"
- moved on the sheet: C1, J5, R13, R14, R15, R16, U4

Commit message: create separate project for IO board
Parts:
- removed D1: D, Diode_THT:D_DO-15_P12.70mm_Horizontal, symbol Device:D
- removed J1: Barrel_Jack_Switch, Connector_BarrelJack:BarrelJack_Horizontal, symbol Connector:Barrel_Jack_Switch
- removed U8: ATmega48-20A, Package_QFP:TQFP-32_7x7mm_P0.8mm, symbol MCU_Microchip_ATmega:ATmega48-20A
- added C10: 100nF, Capacitor_SMD:C_0805_2012Metric_Pad1.18x1.45mm_HandSolder, symbol Device:C
- added D1: D_Schottky, Diode_SMD:D_SOD-123F, symbol Device:D_Schottky
- added J1: Screw_Terminal_01x02, TerminalBlock_Phoenix:TerminalBlock_Phoenix_MKDS-3-2-5.08_1x02_P5.08mm_Horizontal, symbol Connector:Screw_Terminal_01x02
- added J16: Conn_01x05, Connector_Molex:Molex_KK-254_AE-6410-05A_1x05_P2.54mm_Vertical, symbol Connector_Generic:Conn_01x05
- added U6: ATmega328P-A, Package_QFP:TQFP-32_7x7mm_P0.8mm, symbol MCU_Microchip_ATmega:ATmega328P-A
- BZ1: footprint Buzzer_Beeper:MagneticBuzzer_ProSignal_ABT-410-RC -> Connector_Molex:Molex_KK-254_AE-6410-02A_1x02_P2.54mm_Vertical
- C2, C3, C4, C5, C6, C7, C9: footprint (none) -> Capacitor_SMD:C_0805_2012Metric_Pad1.18x1.45mm_HandSolder
- C8: footprint (none) -> Capacitor_SMD:C_1206_3216Metric_Pad1.33x1.80mm_HandSolder
- J2: footprint (none) -> Connector_PinHeader_2.54mm:PinHeader_2x03_P2.54mm_Vertical
- Y1: footprint (none) -> Crystal:Crystal_SMD_HC49-SD_HandSoldering
Connections:
- net UIPanel_BUTT4A is gone; now on net UIPanel_BUTT4A__UIPanel_Prog_MOSI: R26.2, SW9.2
- net UIPanel_BUTT5A is gone; now on net UIPanel_BUTT5A__UIPanel_Prog_MISO: R27.2, SW10.2
- net UIPanel_BUTT6A is gone; now on net UIPanel_BUTT6A__UIPanel_Prog_SCK: R28.2, SW11.2
- net +15V: now also J1.2 (Pin_2)
- net +5V: now also PS1.4 (Vout)
- net GND: no longer BZ1.2 (-)
- net GNDPWR: now also SW1.3 (C), J1.1 (Pin_1)
- net UIPanel_+5V: now also BZ1.1 (+), D10.1 (K), D11.1 (K), D12.1 (K), D13.1 (K), D2.1 (K), D3.1 (K), D4.1 (K), D5.1 (K), D6.1 (K), D7.1 (K), D8.1 (K), D9.1 (K), SW10.1, SW11.1, SW12.1, SW13.1, SW14.1, SW2.1, SW4.1, SW5.1, SW6.1, SW7.1, SW8.1, SW9.1, C10.1, J16.3 (Pin_3), U6.18 (AVCC), U6.4 (VCC), U6.6 (VCC)
- net UIPanel_ADC1: now also U6.19 (ADC6)
- net UIPanel_ADC2: now also U6.22 (ADC7)
- net UIPanel_BUTT1A: now also U6.12 (PB0)
- net UIPanel_BUTT1B: now also SW4.2, U6.23 (PC0); no longer SW4.1
- net UIPanel_BUTT2A: now also U6.13 (PB1)
- net UIPanel_BUTT2B: now also SW6.2, U6.24 (PC1); no longer SW6.1
- net UIPanel_BUTT3A: now also U6.14 (PB2)
- net UIPanel_BUTT3B: now also SW8.2, U6.25 (PC2); no longer SW8.1
- net UIPanel_BUTT4A__UIPanel_Prog_MOSI: now also U6.15 (PB3)
- net UIPanel_BUTT4B: now also SW12.2, U6.26 (PC3); no longer SW12.1
- net UIPanel_BUTT5A__UIPanel_Prog_MISO: now also U6.16 (PB4)
- net UIPanel_BUTT5B: now also SW13.2, U6.2 (PD4); no longer SW13.1
- net UIPanel_BUTT6A__UIPanel_Prog_SCK: now also U6.17 (PB5)
- net UIPanel_BUTT6B: now also SW14.2, U6.9 (PD5); no longer SW14.1
- net UIPanel_Enc_A: now also J16.1 (Pin_1), U6.32 (PD2)
- net UIPanel_Enc_B: now also J16.2 (Pin_2), U6.1 (PD3)
- net UIPanel_Enc_BUTT: now also C10.2, J16.5 (Pin_5), U6.10 (PD6)
- net UIPanel_GND: now also J16.4 (Pin_4), U6.21 (GND), U6.3 (GND), U6.5 (GND)
- net UIPanel_RX: now also U6.30 (PD0)
- net UIPanel_SCL: now also U6.28 (PC5)
- net UIPanel_SDA: now also U6.27 (PC4)
- net UIPanel_TX: now also U6.31 (PD1)
- net UIPanel_reset: now also U6.29 (~{RESET}/PC6)
- net XTAL1: now also U6.7 (XTAL1/PB6)
- net XTAL2: now also U6.8 (XTAL2/PB7)
- net at SW1.2 (B), SW15.1 (A): now also D1.2 (A); no longer PS1.1 (Vin)
- net at C9.1: now also U6.20 (AREF)
- new net: BZ1.2 (-), U6.11 (PD7)
- new net: D1.1 (K), PS1.1 (Vin)
Other:
- note added: "(forrás: https://electronics.stackexchange.com/questions/87157/i2c-over-gpio-level-shifter)"
- note removed: "Ez hogy is működik? (forrás: https://electronics.stackexchange.com/questions/87157/i2c-over-gpio-level-shifter)"
- moved on the sheet: BZ1, C6, C7, J4, J5, Q3A, Q3B, R13, R14, R15, R16, R32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

Commit message: Fixed level shifting, power input protection, buzzer drive and UI buttons
Parts:
- removed Q3: FDG6335N, Package_TO_SOT_SMD:SOT-363_SC-70-6, symbol Transistor_FET:FDG6335N
- removed R10, R12, R4, R40, R44, R45, R49, R50, R51, R6, R8: 390, Resistor_SMD:R_0805_2012Metric_Pad1.20x1.40mm_HandSolder, symbol Device:R
- removed R11, R17, R18, R39, R46, R47, R48, R5, R7, R9: 180, Resistor_SMD:R_0805_2012Metric_Pad1.20x1.40mm_HandSolder, symbol Device:R
- removed R13, R14, R15, R16: 10k, Resistor_SMD:R_0805_2012Metric_Pad1.20x1.40mm_HandSolder, symbol Device:R
- added D18: D, symbol Device:D
- added D19: SMAJ12A, Diode_SMD:D_SMA, symbol Diode:SMAJ12A
- added F1: 30R500UF, symbol Device:Polyfuse
- added Q1: 2N7002, Package_TO_SOT_SMD:SOT-23, symbol Transistor_FET:2N7002
- added U7, U8: SN74LV1T34DBV, Package_TO_SOT_SMD:SOT-23-5, symbol Logic_LevelTranslator:SN74LV1T34DBV
- added U9: 4504, symbol 4xxx:4504
- R1: value 180 -> 160; footprint Resistor_SMD:R_0805_2012Metric_Pad1.20x1.40mm_HandSolder -> (none)
- R2: value 390 -> 160; footprint Resistor_SMD:R_0805_2012Metric_Pad1.20x1.40mm_HandSolder -> (none)
- R3: value 180 -> 100k; footprint Resistor_SMD:R_0805_2012Metric_Pad1.20x1.40mm_HandSolder -> (none)
Connections:
- net Mot3_ENC_IN is gone; now on net Mot3_ENC: J14.14 (Pin_14)
- net Mot4_ENC_IN is gone; now on net Mot4_ENC: J14.17 (Pin_17)
- net Mot5_ENC_IN is gone; now on net Mot5_ENC: J14.21 (Pin_21)
- net Mot6_ENC_IN is gone; now on net Mot6_ENC: J14.25 (Pin_25)
- net +15V: now also D19.1 (A1), F1.2; no longer J1.2 (Pin_2)
- net +3V3: now also U8.5 (VCC), U9.16 (VDD)
- net +5V: now also U7.5 (VCC), U9.1 (VCC)
- net GND: now also U7.3 (GND), U8.3 (GND), U9.13 (Select), U9.8 (VSS); no longer R2.1
- net GNDPWR: now also D19.2 (A2)
- net Mot1_ENC: now also J14.4 (Pin_4); no longer R1.2, R2.2
- net Mot2_ENC: now also J14.8 (Pin_8); no longer R3.2
- net UIPanel_+5V: now also R2.2; no longer BZ1.1 (+), D10.1 (K), D11.1 (K), D12.1 (K), D13.1 (K), D2.1 (K), D3.1 (K), D4.1 (K), D5.1 (K), D6.1 (K), D7.1 (K), D8.1 (K), D9.1 (K), SW10.1, SW11.1, SW12.1, SW13.1, SW14.1, SW2.1, SW4.1, SW5.1, SW6.1, SW7.1, SW8.1, SW9.1
- net UIPanel_GND: now also R3.2, Q1.2 (S)
- net UI_RX_3v3: now also U8.4 (Y)
- net UI_RX_5v: now also U8.2 (A)
- net UI_TX_3v3: now also U7.2 (A)
- net UI_TX_5v: now also U7.4 (Y)
- net at BZ1.2 (-): now also D18.2 (A), Q1.3 (D); no longer U6.11 (PD7)
- net Mot1_ENC_IN renamed UIPanel_Buzz
- net UIPanel_Buzz: now also U6.11 (PD7); no longer J14.4 (Pin_4)
- net Mot2_ENC_IN: no longer names the net of R3.1
- net Mot2_ENC_IN: now also R1.2, Q1.1 (G); no longer J14.8 (Pin_8)
- new net: D12.1 (K), SW13.1
- new net: BZ1.1 (+), D18.1 (K), R2.1
- new net: D7.1 (K), SW8.1
- new net: D2.1 (K), SW2.1
- new net: D9.1 (K), SW10.1
- new net: D10.1 (K), SW11.1
- new net: D4.1 (K), SW5.1
- new net: D5.1 (K), SW6.1
- new net: D6.1 (K), SW7.1
- new net: D8.1 (K), SW9.1
- new net: D3.1 (K), SW4.1
- new net: F1.1, J1.2 (Pin_2)
- new net: D11.1 (K), SW12.1
- new net: D13.1 (K), SW14.1
Other:
- note added: "Motor limitswitches level shifting"
- note removed: "(forrás: https://electronics.stackexchange.com/questions/87157/i2c-over-gpio-level-shifter)"
- note removed: "Motor encoder level shifting"
- note removed: "Mérés alapján csak 2V vagy 3V-ig megy fel a fesz -> lehet nem is kell az egész? Miért lehet h csak eddig megy?"
- moved on the sheet: BZ1, C2, C3, C4, C5, C8, C9, D1, D14, J1, J2, PS1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

Commit message: Added limit switches to schematic
Parts:
- added R4, R5, R6, R7, R8, R9: 10k, Resistor_THT:R_Axial_DIN0207_L6.3mm_D2.5mm_P15.24mm_Horizontal, symbol Device:R
- added SW17, SW18, SW19, SW20, SW21, SW22, SW23, SW24, SW25, SW26, SW27, SW28: SW_SPDT, symbol Switch:SW_SPDT
- C10, C6, C7: value 100nF -> 10nF
Connections:
- net +5V: now also R4.1, R5.1, R6.1, R7.1, R8.1, R9.1
- net GND: now also SW17.3 (C), SW18.3 (C), SW19.3 (C), SW20.3 (C), SW21.3 (C), SW22.3 (C), SW23.3 (C), SW24.3 (C), SW25.3 (C), SW26.3 (C), SW27.3 (C), SW28.3 (C)
- net Mot1_LIMIT: now also U9.2 (Aout)
- net Mot1_LIMIT_IN: now also U9.3 (Ain), R4.2, SW17.2 (B), SW18.2 (B)
- net Mot2_LIMIT: now also U9.4 (Bout)
- net Mot2_LIMIT_IN: now also U9.5 (Bin), R5.2, SW19.2 (B), SW20.2 (B)
- net Mot3_LIMIT: now also U9.6 (Cout)
- net Mot3_LIMIT_IN: now also U9.7 (Cin), R6.2, SW21.2 (B), SW22.2 (B)
- net Mot4_LIMIT: now also U9.10 (Dout)
- net Mot4_LIMIT_IN: now also U9.9 (Din), R7.2, SW23.2 (B), SW26.2 (B)
- net Mot5_LIMIT: now also U9.12 (Eout)
- net Mot5_LIMIT_IN: now also U9.11 (Ein), R8.2, SW24.2 (B), SW27.2 (B)
- net Mot6_LIMIT: now also U9.15 (Fout)
- net Mot6_LIMIT_IN: now also U9.14 (Fin), R9.2, SW25.2 (B), SW28.2 (B)
- no-connect marks 2 -> 14
Other:
- note added: "Motor limitswitches (have been modified on the robotarm)"
- moved on the sheet: R41, R42, R43, U1, U2, U3, U9

Commit message: Split control board and I/O cards into separate projects
Parts:
- removed BZ1: Buzzer, Connector_Molex:Molex_KK-254_AE-6410-02A_1x02_P2.54mm_Vertical, symbol Device:Buzzer
- removed C10, C6, C7: 10nF, Capacitor_SMD:C_0805_2012Metric_Pad1.18x1.45mm_HandSolder, symbol Device:C
- removed C2, C3: 22pF, Capacitor_SMD:C_0805_2012Metric_Pad1.18x1.45mm_HandSolder, symbol Device:C
- removed C4, C5: 1uF, Capacitor_SMD:C_0805_2012Metric_Pad1.18x1.45mm_HandSolder, symbol Device:C
- removed C8: 4.7uF, Capacitor_SMD:C_1206_3216Metric_Pad1.33x1.80mm_HandSolder, symbol Device:C_Polarized
- removed C9: 100nF, Capacitor_SMD:C_0805_2012Metric_Pad1.18x1.45mm_HandSolder, symbol Device:C
- removed D10, D11, D12, D13, D14, D2, D3, D4, D5, D6, D7, D8, D9: LED, LED_THT:LED_D5.0mm, symbol Device:LED
- removed D18: D, symbol Device:D
- removed J10, J11, J12, J13, J7, J9: Conn_01x06, Connector_Molex:Molex_KK-254_AE-6410-06A_1x06_P2.54mm_Vertical, symbol Connector_Generic:Conn_01x06
- removed J15, J3: Conn_01x03, Connector_Molex:Molex_KK-254_AE-6410-03A_1x03_P2.54mm_Vertical, symbol Connector_Generic:Conn_01x03
- removed J16: Conn_01x05, Connector_Molex:Molex_KK-254_AE-6410-05A_1x05_P2.54mm_Vertical, symbol Connector_Generic:Conn_01x05
- removed J2: Conn_02x03_Counter_Clockwise, Connector_PinHeader_2.54mm:PinHeader_2x03_P2.54mm_Vertical, symbol Connector_Generic:Conn_02x03_Counter_Clockwise
- removed J4, J5: Conn_01x04, Connector_Molex:Molex_KK-254_AE-6410-04A_1x04_P2.54mm_Vertical, symbol Connector_Generic:Conn_01x04
- removed J6: Conn_02x13_Top_Bottom, Connector_IDC:IDC-Header_2x13_P2.54mm_Vertical, symbol Connector_Generic:Conn_02x13_Top_Bottom
- removed Q1: 2N7002, Package_TO_SOT_SMD:SOT-23, symbol Transistor_FET:2N7002
- removed R1, R2: 160, symbol Device:R
- removed R20, R21, R22, R23, R24, R25, R26, R27, R28, R29, R30, R31, R35: 220, Resistor_SMD:R_0805_2012Metric_Pad1.20x1.40mm_HandSolder, symbol Device:R
- removed R3: 100k, symbol Device:R
- removed R32, R33, R34, R52: 10k, Resistor_SMD:R_0805_2012Metric_Pad1.20x1.40mm_HandSolder, symbol Device:R
- removed SW10, SW11, SW12, SW13, SW14, SW16, SW2, SW4, SW5, SW6, SW7, SW8, SW9: SW_Push, Connector_Molex:Molex_KK-254_AE-6410-02A_1x02_P2.54mm_Vertical, symbol Switch:SW_Push
- removed SW3: RotaryEncoder_Switch, IIT_5dof_arm:Molex_for_encoder_1x05_P2.54mm_Vertical, symbol Device:RotaryEncoder_Switch
- removed U6: ATmega328P-A, Package_QFP:TQFP-32_7x7mm_P0.8mm, symbol MCU_Microchip_ATmega:ATmega328P-A
- removed Y1: 16MHz, Crystal:Crystal_SMD_HC49-SD_HandSoldering, symbol Device:Crystal
- D19: footprint Diode_SMD:D_SMA -> Diode_SMD:D_SMA_Handsoldering
- F1: footprint (none) -> Capacitor_THT:C_Rect_L13.5mm_W4.0mm_P10.00mm_FKS3_FKP3_MKS4
- U7, U8: footprint Package_TO_SOT_SMD:SOT-23-5 -> Package_TO_SOT_SMD:SOT-23-5_HandSoldering
- U9: footprint (none) -> Package_DIP:DIP-16_W7.62mm_Socket_LongPads
Connections:
- net +5V: now also J14.3 (Pin_3); no longer J14.13 (Pin_13)
- net Mot1_LIMIT: now also U5.7 (P3); no longer U5.4 (P0)
- net Mot1_LIMIT_IN: now also J14.15 (Pin_15); no longer J14.5 (Pin_5)
- net Mot1_OUT1: now also J14.14 (Pin_14); no longer J14.2 (Pin_2)
- net Mot1_OUT2: now also J14.16 (Pin_16); no longer J14.3 (Pin_3)
- net Mot2_ENC: now also J14.2 (Pin_2); no longer J14.8 (Pin_8)
- net Mot2_LIMIT: now also U5.6 (P2); no longer U5.5 (P1)
- net Mot2_LIMIT_IN: now also J14.13 (Pin_13); no longer J14.9 (Pin_9)
- net Mot2_OUT1: now also J14.18 (Pin_18); no longer J14.6 (Pin_6)
- net Mot2_OUT2: now also J14.20 (Pin_20); no longer J14.7 (Pin_7)
- net Mot3_ENC: now also J14.8 (Pin_8); no longer J14.14 (Pin_14)
- net Mot3_LIMIT: now also U5.12 (P7); no longer U5.6 (P2)
- net Mot3_LIMIT_IN: now also J14.11 (Pin_11); no longer J14.10 (Pin_10)
- net Mot3_OUT1: now also J14.23 (Pin_23); no longer J14.11 (Pin_11)
- net Mot3_OUT2: now also J14.21 (Pin_21); no longer J14.12 (Pin_12)
- net Mot4_ENC: now also J14.6 (Pin_6); no longer J14.17 (Pin_17)
- net Mot4_LIMIT: now also U5.11 (P6); no longer U5.7 (P3)
- net Mot4_LIMIT_IN: now also J14.5 (Pin_5); no longer J14.18 (Pin_18)
- net Mot4_OUT1: now also J14.19 (Pin_19); no longer J14.15 (Pin_15)
- net Mot4_OUT2: now also J14.17 (Pin_17); no longer J14.16 (Pin_16)
- net Mot5_ENC: now also J14.12 (Pin_12); no longer J14.21 (Pin_21)
- net Mot5_LIMIT: now also U5.10 (P5); no longer U5.9 (P4)
- net Mot5_LIMIT_IN: now also J14.7 (Pin_7); no longer J14.22 (Pin_22)
- net Mot5_OUT1: now also J14.22 (Pin_22); no longer J14.19 (Pin_19)
- net Mot5_OUT2: now also J14.24 (Pin_24); no longer J14.20 (Pin_20)
- net Mot6_ENC: now also J14.10 (Pin_10); no longer J14.25 (Pin_25)
- net Mot6_LIMIT: now also U5.9 (P4); no longer U5.10 (P5)
- net Mot6_LIMIT_IN: now also J14.9 (Pin_9); no longer J14.26 (Pin_26)
- net Mot6_OUT1: now also J14.26 (Pin_26); no longer J14.23 (Pin_23)
- net Mot6_OUT2: now also J14.25 (Pin_25); no longer J14.24 (Pin_24)
- net mot1_A: now also U4.12 (GPIO14/ADC16/TOUCH6/SPI-CLK); no longer U4.25 (GPIO0/ADC11/TOUCH1)
- net mot1_B: now also U4.11 (GPIO27/ADC17/TOUCH7); no longer U4.24 (GPIO2/ADC12/TOUCH2)
- net mot2_A: now also U4.10 (GPIO26/ADC19/DAC2); no longer U4.12 (GPIO14/ADC16/TOUCH6/SPI-CLK)
- net mot2_B: now also U4.9 (GPIO25/ADC18/DAC1); no longer U4.23 (GPIO15/ADC13/TOUCH3)
- net mot3_A: now also U4.37 (GPIO23/VSPI-MOSI); no longer U4.11 (GPIO27/ADC17/TOUCH7)
- net mot3_B: now also U4.31 (GPIO19/VSPI-MISO); no longer U4.26 (GPIO4/ADC10/TOUCH0)
- net mot4_A: now also U4.30 (GPIO18/VSPI-SCK); no longer U4.29 (GPIO5/VSPI-SS)
- net mot4_B: now also U4.29 (GPIO5/VSPI-SS); no longer U4.10 (GPIO26/ADC19/DAC2)
- net mot5_A: now also U4.26 (GPIO4/ADC10/TOUCH0); no longer U4.31 (GPIO19/VSPI-MISO)
- net mot5_B: now also U4.25 (GPIO0/ADC11/TOUCH1); no longer U4.30 (GPIO18/VSPI-SCK)
- net mot6_A: now also U4.24 (GPIO2/ADC12/TOUCH2); no longer U4.13 (GPIO12/ADC15/TOUCH5/SPI-MISO)
- net mot6_B: now also U4.23 (GPIO15/ADC13/TOUCH3); no longer U4.37 (GPIO23/VSPI-MOSI)
- net ~{Fault}_12: now also U4.13 (GPIO12/ADC15/TOUCH5/SPI-MISO); no longer U4.9 (GPIO25/ADC18/DAC1)
- net ~{Fault}_34: now also U5.5 (P1); no longer U5.11 (P6)
- net ~{Fault}_56: now also U5.4 (P0); no longer U5.12 (P7)
Other:
- note added: "Port extension Limit switch inputs & motor faults"
- note removed: "Port expanding"
- note removed: "Programming with: https://github.com/MCUdude/MiniCore"
- note removed: "Robot arm interface panel"
- note removed: "User interface panel"
- moved on the sheet: C1, D15, D16, D17, J14, J8, R19, R36, R37, R38, R4, R41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

Commit message: Change motor power LED footprint to connector
Parts:
- D15: footprint LED_THT:LED_D5.0mm -> Connector_Molex:Molex_KK-254_AE-6410-02A_1x02_P2.54mm_Vertical
Changed lines of the file:
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@@
 			)
 		)
-		(property "Footprint" "LED_THT:LED_D5.0mm"
+		(property "Footprint" "Connector_Molex:Molex_KK-254_AE-6410-02A_1x02_P2.54mm_Vertical"
 			(at 124.46 30.48 0)
 			(effects
