File: PCB/IIT_5dof_arm/IIT_5dof_arm.kicad_sch (KiCad schematic)
At the start: 61 parts, among them J1 Screw_Terminal_01x02, J2 Conn_01x06, J3 Conn_01x06, J4 Conn_01x06, J5 Conn_01x06, J6 Conn_01x06, J7 Conn_01x06, J9 DE9_Receptacle_MountingHoles, SW1 SW_MAIN, SW15 SW_MOT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

Commit message: Extend ESD protection on RS-232 interface and tidy up schematic
Parts:
- added D5: SMAJ12A, Diode_SMD:D_SMA_Handsoldering, symbol Diode:SMAJ12A
Connections:
- net +5V: now also D5.1 (A1)
- net GND: now also D5.2 (A2)
Other:
- note added: "Logic power feedback LED"
- note added: "PCB mounting"
- note added: "UART TTL to RS-232"
- note removed: "UART level shifting"
- moved on the sheet: C1, C2, C3, C4, C5, C6, D1, D15, D19, D2, D3, D4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
