File: PCB/IIT_5dof_arm_IO/IIT_5dof_arm_IO.kicad_sch (KiCad schematic)
At the start: 138 parts, among them J1 Conn_01x05, J10 Conn_01x02, J11 Conn_01x02, J12 Conn_01x02, J13 Conn_01x02, J14 Conn_01x02, J15 Conn_01x02, J16 Conn_01x02, J17 Conn_01x02, J18 Conn_01x02, J19 Conn_01x02, J2 Conn_01x03, J20 Conn_01x02, J21 Conn_01x02, J22 Conn_01x02, J23 Conn_01x02, J24 Conn_01x02, J25 Conn_01x02, J26 Conn_01x02, J27 Conn_01x02, J28 Conn_01x02, J3 Conn_02x03_Odd_Even, J4 Conn_01x02, J5 Conn_01x04, J6 DE9_Plug_MountingHoles, J7 Conn_01x02, J8 Conn_01x04, J9 Conn_01x02, Q1 2N7002, Q2 BSS84, Q3 BSS84, Q4 BSS84, SW1 SW_Push, SW10 SW_Push, SW11 SW_Push, SW12 SW_Push, SW13 SW_Push, SW14 SW_Push, SW15 SW_SPDT, SW16 SW_Push, SW2 SW_Push, SW3 SW_Push, SW4 SW_Push, SW5 SW_Push, SW6 SW_Push, SW7 RotaryEncoder_Switch, SW8 SW_Push, SW9 SW_Push, U1 ATmega328P-A, U2 MAX3232, Y1 16MHz

Commit message: Organize schematic
Parts:
- added J29, J30, J31, J32, J33, J34: Conn_01x02, Connector_Molex:Molex_KK-254_AE-6410-04A_1x04_P2.54mm_Vertical, symbol Connector_Generic:Conn_01x02
- J3: footprint (none) -> Connector_IDC:IDC-Header_2x03_P2.54mm_Vertical
Connections:
- net UIPanel_ADC2 is gone; now on net ToggleMotors: J4.1 (Pin_1)
- net UIPanel_+5V: now also J12.1 (Pin_1), J23.1 (Pin_1), J24.1 (Pin_1), J25.1 (Pin_1), J26.1 (Pin_1), J9.1 (Pin_1), J30.1 (Pin_1), J31.1 (Pin_1), J32.1 (Pin_1)
- net UIPanel_BUTT1A: now also J14.1 (Pin_1)
- net UIPanel_BUTT1B: now also J15.1 (Pin_1)
- net UIPanel_BUTT2A: now also J13.1 (Pin_1)
- net UIPanel_BUTT2B: now also J16.1 (Pin_1)
- net UIPanel_BUTT3A: now also J33.1 (Pin_1)
- net UIPanel_BUTT3B: now also J17.1 (Pin_1)
- net UIPanel_BUTT4A: now also J11.1 (Pin_1)
- net UIPanel_BUTT4B: now also J18.1 (Pin_1)
- net UIPanel_BUTT5A: now also J10.1 (Pin_1)
- net UIPanel_BUTT5B__UIPanel_Prog_SCK: now also J19.1 (Pin_1)
- net UIPanel_BUTT6A__UIPanel_Prog_MOSI: now also J20.1 (Pin_1)
- net UIPanel_BUTT6B__UIPanel_Prog_MISO: now also J21.1 (Pin_1)
- net UIPanel_GND: now also C1.1, J10.2 (Pin_2), J11.2 (Pin_2), J13.2 (Pin_2), J14.2 (Pin_2), J15.2 (Pin_2), J16.2 (Pin_2), J17.2 (Pin_2), J18.2 (Pin_2), J19.2 (Pin_2), J20.2 (Pin_2), J21.2 (Pin_2), J33.2 (Pin_2); no longer C1.2
- net at D2.1 (K), R4.1: now also J25.2 (Pin_2)
- net at D7.1 (K), R9.1: now also J32.2 (Pin_2)
- net at D6.1 (K), R8.1: now also J27.2 (Pin_2)
- net at D6.2 (A), Q3.3 (D), R29.1: now also J27.1 (Pin_1)
- net at J24.2 (Pin_2): now also D3.1 (K), R5.1
- net at D11.1 (K), R13.1: now also J29.2 (Pin_2)
- net at J23.2 (Pin_2): now also D4.1 (K), R6.1
- net at U1.20 (AREF): now also C1.2; no longer C1.1
- net at BZ1.1 (+), D13.1 (K), R19.1: now also J34.1 (Pin_1)
- net at BZ1.2 (-), D13.2 (A), Q1.3 (D): now also J34.2 (Pin_2)
- net at D12.2 (A), Q4.3 (D), R35.1: now also J28.1 (Pin_1)
- net at D5.1 (K), R7.1: now also J9.2 (Pin_2)
- net at D12.1 (K), R14.1: now also J28.2 (Pin_2)
- net at D8.1 (K), R10.1: now also J31.2 (Pin_2)
- net at D10.1 (K), R12.1: now also J30.2 (Pin_2)
- net at D9.1 (K), R11.1: now also J12.2 (Pin_2)
- net at J26.2 (Pin_2): now also D1.1 (K), R3.1
- net at D11.2 (A), Q2.3 (D), R34.1: now also J29.1 (Pin_1)
- net 5V_LED-: no longer names the net of D14.1 (K), J22.2 (Pin_2), R20.1
- net UIPanel_ADC1 renamed PotmeterInput
Other:
- note added: "Motor toggle connection"
- note added: "Potentiometer connection"
- moved on the sheet: C1, C15, C16, C17, C18, C19, C20, C21, C22, C23, C24, C25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
